Commit message: kopa noviniek

File: waver-humble/waver_description/urdf/imu.xacro (robot description, xacro)
@@ -4,4 +4,10 @@
     <xacro:include filename="$(find waver_description)/urdf/util.xacro" />
     <link name="imu_link">
+        <inertial>
+            <mass value="0.010" />
+            <origin xyz="0 0 0" rpy="0 0 0" />
+            <inertia ixx="3.4e-7" iyy="3.4e-7" izz="6.7e-7"
+                     ixy="0" ixz="0" iyz="0" />
+        </inertial>
         <visual>
             <origin xyz="${position_imu}" rpy="0 0 ${pi/2}" />
@@ -17,4 +23,8 @@
         <child link="imu_link" />
     </joint>
+    <!-- Prevent Gazebo Harmonic from lumping this fixed joint into base_footprint -->
+    <gazebo reference="top_imu_joint">
+        <preserveFixedJoint>true</preserveFixedJoint>
+    </gazebo>
     <gazebo reference="imu_link">
         <material>Gazebo/Orange</material>
@@ -23,6 +33,19 @@
             <always_on>true</always_on>
             <update_rate>100</update_rate>
-            <visualize>true</visualize>
+            <visualize>false</visualize>
             <topic>imu</topic>
+            <gz_frame_id>imu_link</gz_frame_id>
+            <imu>
+                <angular_velocity>
+                    <x><noise type="gaussian"><mean>0</mean><stddev>2e-4</stddev></noise></x>
+                    <y><noise type="gaussian"><mean>0</mean><stddev>2e-4</stddev></noise></y>
+                    <z><noise type="gaussian"><mean>0</mean><stddev>2e-4</stddev></noise></z>
+                </angular_velocity>
+                <linear_acceleration>
+                    <x><noise type="gaussian"><mean>0</mean><stddev>1.7e-2</stddev></noise></x>
+                    <y><noise type="gaussian"><mean>0</mean><stddev>1.7e-2</stddev></noise></y>
+                    <z><noise type="gaussian"><mean>0</mean><stddev>1.7e-2</stddev></noise></z>
+                </linear_acceleration>
+            </imu>
         </sensor>
     </gazebo>

File: waver-humble/waver_description/urdf/lidar.xacro (robot description, xacro)
@@ -28,4 +28,8 @@
         <child link="lidar_link" />
     </joint>
+    <!-- Prevent Gazebo Harmonic from lumping this fixed joint into base_footprint -->
+    <gazebo reference="lidar_joint">
+        <preserveFixedJoint>true</preserveFixedJoint>
+    </gazebo>
     <gazebo reference="lidar_link">
         <material>Gazebo/Black</material>

File: waver-humble/waver_description/urdf/rasp_pi_camera.xacro (robot description, xacro)
@@ -4,4 +4,10 @@
     <xacro:include filename="$(find waver_description)/urdf/util.xacro" />
     <link name="rasp_pi_camera_link">
+        <inertial>
+            <mass value="${rasp_pi_camera_mass}" />
+            <origin xyz="0 0 0" rpy="0 0 0" />
+            <inertia ixx="1.7e-7" iyy="1.8e-7" izz="3.0e-7"
+                     ixy="0" ixz="0" iyz="0" />
+        </inertial>
         <visual>
             <origin xyz="0 0.0125 0" rpy="0 0 ${-pi/2}" />
@@ -24,4 +30,8 @@
         <child link="rasp_pi_camera_link" />
     </joint>
+    <!-- Prevent Gazebo Harmonic from lumping this fixed joint into base_footprint -->
+    <gazebo reference="rasp_pi_camera_joint">
+        <preserveFixedJoint>true</preserveFixedJoint>
+    </gazebo>
     <gazebo reference="rasp_pi_camera_link">
         <material>Gazebo/Black</material>

File: waver-humble/waver_description/urdf/waver.gazebo.xacro (robot description, xacro)
@@ -40,5 +40,5 @@
   <gazebo reference="wheel_back_left_link">
     <mu1>0.8</mu1>
-    <mu2>0.8</mu2>
+    <mu2>0.05</mu2>
     <selfCollide>false</selfCollide>
     <material>Gazebo/Black</material>
@@ -46,5 +46,5 @@
   <gazebo reference="wheel_front_left_link">
     <mu1>0.8</mu1>
-    <mu2>0.8</mu2>
+    <mu2>0.05</mu2>
     <selfCollide>false</selfCollide>
     <material>Gazebo/Black</material>
@@ -52,5 +52,5 @@
   <gazebo reference="wheel_front_right_link">
     <mu1>0.8</mu1>
-    <mu2>0.8</mu2>
+    <mu2>0.05</mu2>
     <selfCollide>false</selfCollide>
     <material>Gazebo/Black</material>
@@ -58,34 +58,37 @@
   <gazebo reference="wheel_back_right_link">
     <mu1>0.8</mu1>
-    <mu2>0.8</mu2>
+    <mu2>0.05</mu2>
     <selfCollide>false</selfCollide>
     <material>Gazebo/Black</material>
   </gazebo>
   <gazebo>
-    <plugin filename="libgz-sim-diff-drive-system.so" name="gz::sim::systems::DiffDrive">
-      <left_joint>wheel_front_left_joint</left_joint>
-      <right_joint>wheel_front_right_joint</right_joint>
-      <left_joint>wheel_back_left_joint</left_joint>
-      <right_joint>wheel_back_right_joint</right_joint>
+    <!-- 4-wheel skid-steer, front+rear on each side share the same drive command -->
+    <plugin filename="gz-sim-diff-drive-system" name="gz::sim::systems::DiffDrive">
+      <left_joint>wheel_front_left_link_joint</left_joint>
+      <right_joint>wheel_front_right_link_joint</right_joint>
+      <left_joint>wheel_back_left_link_joint</left_joint>
+      <right_joint>wheel_back_right_link_joint</right_joint>
       <wheel_separation>${wheel_separation}</wheel_separation>
       <wheel_radius>${wheel_radius}</wheel_radius>
-      <max_linear_acceleration>2.0</max_linear_acceleration>
-      <min_linear_acceleration>-2.0</min_linear_acceleration>
-      <max_angular_acceleration>4.0</max_angular_acceleration>
-      <min_angular_acceleration>-4.0</min_angular_acceleration>
+      <max_linear_acceleration>1.5</max_linear_acceleration>
+      <min_linear_acceleration>-1.5</min_linear_acceleration>
+      <max_angular_acceleration>3.0</max_angular_acceleration>
+      <min_angular_acceleration>-3.0</min_angular_acceleration>
+      <max_linear_velocity>0.35</max_linear_velocity>
+      <min_linear_velocity>-0.35</min_linear_velocity>
+      <max_angular_velocity>1.5</max_angular_velocity>
+      <min_angular_velocity>-1.5</min_angular_velocity>
       <topic>cmd_vel</topic>
       <odom_topic>odometry</odom_topic>
-      <tf_topic>tf</tf_topic>
+      <tf_topic>/tf</tf_topic>
       <frame_id>odom</frame_id>
       <child_frame_id>base_footprint</child_frame_id>
       <odom_publish_frequency>30</odom_publish_frequency>
     </plugin>
-    <plugin filename="libgz-sim-joint-state-publisher-system.so"
+    <plugin filename="gz-sim-joint-state-publisher-system"
       name="gz::sim::systems::JointStatePublisher">
       <topic>joint_states</topic>
     </plugin>
-    <plugin filename="libgz-sim-sensors-system.so" name="gz::sim::systems::Sensors">
-      <render_engine>ogre2</render_engine>
-    </plugin>
+    <!-- Sensors and Imu plugins belong in the world SDF waver_gazebo worlds not on this model. -->
   </gazebo>
 </robot>

File: waver-humble/waver_description/urdf/waver.xacro (robot description, xacro)
@@ -1,239 +1,280 @@
 <?xml version="1.0"?>
 <robot name="waver" xmlns:xacro="http://www.ros.org/wiki/xacro">
-  <xacro:arg name="sim_control" default="gazebo" />
-  <xacro:arg name="camera_type" default="raspi" />
-  <xacro:include filename="$(find waver_description)/urdf/materials.xacro" />
+  <xacro:arg name="sim_control"  default="gazebo" />
+  <xacro:arg name="camera_type" default="raspi"  />
   <xacro:include filename="$(find waver_description)/urdf/util.xacro" />
-  <xacro:include filename="$(find waver_description)/urdf/lidar.xacro" />
-  <xacro:include filename="$(find waver_description)/urdf/imu.xacro" />
-  <!-- ************************** Simulation Control ************************** -->
   <xacro:if value="${'$(arg sim_control)' == 'gazebo'}">
     <xacro:include filename="$(find waver_description)/urdf/waver.gazebo.xacro" />
   </xacro:if>
-  <xacro:if value="${'$(arg sim_control)' == 'ros2'}">
-    <xacro:include filename="$(find waver_description)/urdf/waver.control.xacro" />
-  </xacro:if>
-  <!-- ***************************** Camera Type ***************************** -->
-  <xacro:if value="${'$(arg camera_type)' == 'raspi'}">
-    <xacro:include filename="$(find waver_description)/urdf/rasp_pi_camera.xacro" />
-  </xacro:if>
-  <xacro:if value="${'$(arg camera_type)' == 'depth'}">
-    <xacro:include filename="$(find waver_description)/urdf/depth_camera_zedxm.xacro" />
-  </xacro:if>
-  <!-- ******************************* Links ******************************* -->
-  <link name="base_footprint"></link>
+  <!-- ── Materials ─────────────────────────────────────────────────── -->
+  <material name="dark_gray"><color rgba="0.13 0.13 0.13 1"/></material>
+  <material name="black">    <color rgba="0.05 0.05 0.05 1"/></material>
+  <material name="gray">     <color rgba="0.55 0.55 0.55 1"/></material>
+  <material name="green">    <color rgba="0.1  0.5  0.1  1"/></material>
+  <material name="blue">     <color rgba="0.1  0.1  0.75 1"/></material>
+  <material name="orange">   <color rgba="0.95 0.45 0.0  1"/></material>
+  <material name="silver">   <color rgba="0.78 0.78 0.78 1"/></material>
+  <!-- ── Chassis dimensions ──────────────────────────────────────────
+       WaveRover real dimensions (from CAD):
+         length 183 mm, width 130 mm, body height 50 mm
+       Top shell plate: 165×118×16 mm flat cover on body
+       Wheels: radius 40.6 mm, width 42.5 mm, separation 123 mm
+  ────────────────────────────────────────────────────────────────── -->
+  <xacro:property name="body_l"  value="0.183"/>
+  <xacro:property name="body_w"  value="0.130"/>
+  <xacro:property name="body_h"  value="0.050"/>
+  <xacro:property name="shell_h" value="0.016"/>
+  <!-- ── base_footprint (virtual ground reference) ──────────────────── -->
+  <link name="base_footprint"/>
+  <joint name="base_joint" type="fixed">
+    <origin xyz="0 0 ${wheel_radius}" rpy="0 0 0"/>
+    <parent link="base_footprint"/>
+    <child  link="base_link"/>
+  </joint>
+  <!-- ── Main chassis body ─────────────────────────────────────────── -->
   <link name="base_link">
     <inertial>
-      <mass value="${mass_base}" />
-      <origin xyz="${mass_center_base}" rpy="0 0 ${pi/2}" />
-      <inertia ixx="0.00024519341275127564" iyy="0.0001572047252476648" izz="0.0001572047252476648"
-        ixy="0.0" iyz="0.0" ixz="0.0" />
+      <mass value="1.2"/>
+      <origin xyz="0 0 0"/>
+      <inertia ixx="0.003" iyy="0.005" izz="0.006"
+               ixy="0" ixz="0" iyz="0"/>
+    </inertial>
+    <!-- main rectangular body box -->
+    <visual name="body">
+      <origin xyz="0 0 0"/>
+      <geometry><box size="${body_l} ${body_w} ${body_h}"/></geometry>
+      <material name="dark_gray"/>
+    </visual>
+    <!-- orange accent stripe on the front face -->
+    <visual name="front_stripe">
+      <origin xyz="${body_l/2 - 0.004} 0 0.006"/>
+      <geometry><box size="0.006 ${body_w - 0.010} 0.010"/></geometry>
+      <material name="orange"/>
+    </visual>
+    <!-- small bumper protrusion at rear -->
+    <visual name="rear_bumper">
+      <origin xyz="${-(body_l/2 + 0.006)} 0 ${-body_h/2 + 0.008}"/>
+      <geometry><box size="0.012 ${body_w + 0.004} 0.016"/></geometry>
+      <material name="black"/>
+    </visual>
+    <collision>
+      <origin xyz="0 0 0"/>
+      <geometry><box size="${body_l} ${body_w} ${body_h}"/></geometry>
+    </collision>
+  </link>
+  <!-- ── Top cover plate (sits on top of chassis) ───────────────────── -->
+  <link name="top_shell_link">
+    <inertial>
+      <mass value="0.050"/>
+      <origin xyz="0 0 0"/>
+      <inertia ixx="1.5e-4" iyy="2.0e-4" izz="3.0e-4"
+               ixy="0" ixz="0" iyz="0"/>
     </inertial>
     <visual>
-      <origin xyz="0 0 0" rpy="0 0 ${pi/2}" />
-      <geometry>
-        <mesh filename="package://waver_description/meshes/base_link.stl" scale="${scale}" />
-      </geometry>
-      <xacro:dark_gray_material />
-    </visual>
-    <collision>
-      <origin xyz="0 0 0" rpy="0 0 ${pi/2}" />
-      <geometry>
-        <mesh filename="package://waver_description/meshes/base_link.stl" scale="${scale}" />
-      </geometry>
-    </collision>
-  </link>
-  <link name="top_shell_link">
-    <inertial>
-      <mass value="${mass_top}" />
-      <origin xyz="${mass_center_top}" rpy="0 0 ${pi/2}" />
-      <inertia ixx="0.0009909748444994777" iyy="0.0008084780487946392" izz="0.0016391807866491105"
-        ixy="0.0" iyz="0.0" ixz="0.0" />
+      <origin xyz="0 0 0"/>
+      <geometry><box size="0.165 0.118 ${shell_h}"/></geometry>
+      <material name="dark_gray"/>
+    </visual>
+    <collision>
+      <origin xyz="0 0 0"/>
+      <geometry><box size="0.165 0.118 ${shell_h}"/></geometry>
+    </collision>
+  </link>
+  <joint name="top_shell_joint" type="fixed">
+    <origin xyz="0 0 ${body_h/2 + shell_h/2}" rpy="0 0 0"/>
+    <parent link="base_link"/>
+    <child  link="top_shell_link"/>
+  </joint>
+  <gazebo reference="top_shell_joint">
+    <preserveFixedJoint>true</preserveFixedJoint>
+  </gazebo>
+  <!-- ── LiDAR LD19  (cylindrical puck on a mounting post) ────────────
+       Joint placed at centre of the puck.
+       Post visual is offset downward inside the same link so it renders
+       as an integrated mounting post below the spinning puck.
+  ────────────────────────────────────────────────────────────────── -->
+  <link name="lidar_link">
+    <inertial>
+      <mass value="0.046"/>
+      <origin xyz="0 0 0"/>
+      <inertia ixx="1.2e-5" iyy="1.5e-5" izz="1.9e-5"
+               ixy="0" ixz="0" iyz="0"/>
+    </inertial>
+    <!-- vertical mounting post (below the puck) -->
+    <visual name="post">
+      <origin xyz="0 0 -0.033"/>
+      <geometry><cylinder radius="0.007" length="0.036"/></geometry>
+      <material name="silver"/>
+    </visual>
+    <!-- LD19 puck housing -->
+    <visual name="puck">
+      <origin xyz="0 0 0"/>
+      <geometry><cylinder radius="0.019" length="0.030"/></geometry>
+      <material name="gray"/>
+    </visual>
+    <collision>
+      <origin xyz="0 0 0"/>
+      <geometry><cylinder radius="0.019" length="0.030"/></geometry>
+    </collision>
+  </link>
+  <!-- z = top of chassis + shell thickness + post height + half puck -->
+  <joint name="lidar_joint" type="fixed">
+    <origin xyz="0.04 0 ${body_h/2 + shell_h + 0.036 + 0.015}" rpy="0 0 0"/>
+    <parent link="base_link"/>
+    <child  link="lidar_link"/>
+  </joint>
+  <gazebo reference="lidar_joint">
+    <preserveFixedJoint>true</preserveFixedJoint>
+  </gazebo>
+  <!-- ── Camera (front face, with PCB board + lens cylinder) ─────────── -->
+  <link name="rasp_pi_camera_link">
+    <inertial>
+      <mass value="0.0035"/>
+      <origin xyz="0 0 0"/>
+      <inertia ixx="1.7e-7" iyy="1.8e-7" izz="3.0e-7"
+               ixy="0" ixz="0" iyz="0"/>
+    </inertial>
+    <!-- PCB board body -->
+    <visual name="board">
+      <origin xyz="0 0 0"/>
+      <geometry><box size="0.010 0.025 0.023"/></geometry>
+      <material name="black"/>
+    </visual>
+    <!-- lens cylinder pointing forward (+x) -->
+    <visual name="lens">
+      <origin xyz="0.007 0 0" rpy="0 ${pi/2} 0"/>
+      <geometry><cylinder radius="0.004" length="0.006"/></geometry>
+      <material name="blue"/>
+    </visual>
+    <collision>
+      <origin xyz="0 0 0"/>
+      <geometry><box size="0.010 0.025 0.023"/></geometry>
+    </collision>
+  </link>
+  <joint name="rasp_pi_camera_joint" type="fixed">
+    <origin xyz="${body_l/2 + 0.005} 0 0.005" rpy="0 0 0"/>
+    <parent link="base_link"/>
+    <child  link="rasp_pi_camera_link"/>
+  </joint>
+  <gazebo reference="rasp_pi_camera_joint">
+    <preserveFixedJoint>true</preserveFixedJoint>
+  </gazebo>
+  <!-- ── IMU (flat chip on top of chassis, hidden under shell) ─────── -->
+  <link name="imu_link">
+    <inertial>
+      <mass value="0.010"/>
+      <origin xyz="0 0 0"/>
+      <inertia ixx="3.4e-7" iyy="3.4e-7" izz="6.7e-7"
+               ixy="0" ixz="0" iyz="0"/>
     </inertial>
     <visual>
-      <origin xyz="0 0 0" rpy="0 0 ${pi/2}" />
-      <geometry>
-        <mesh filename="package://waver_description/meshes/top_shell_link.stl" scale="${scale}" />
-      </geometry>
-      <xacro:dark_gray_material />
-    </visual>
-    <collision>
-      <origin xyz="0 0 0" rpy="0 0 ${pi/2}" />
-      <geometry>
-        <mesh filename="package://waver_description/meshes/top_shell_link.stl" scale="${scale}" />
-      </geometry>
-    </collision>
-  </link>
-  <link name="accessories_link">
-    <visual>
-      <origin xyz="${position_acces}" rpy="0 0 ${pi/2}" />
-      <geometry>
-        <mesh filename="package://waver_description/meshes/accessories_link.stl" scale="${scale}" />
-      </geometry>
-      <xacro:black_material />
-    </visual>
-    <collision>
-      <origin xyz="${position_acces}" rpy="0 0 ${pi/2}" />
-      <geometry>
-        <mesh filename="package://waver_description/meshes/accessories_link.stl" scale="${scale}" />
-      </geometry>
-    </collision>
-  </link>
-  <link name="accessories1_link">
-    <visual>
-      <origin xyz="${position_acces1}" rpy="0 0 ${pi/2}" />
-      <geometry>
-        <mesh filename="package://waver_description/meshes/accessories1_link.stl" scale="${scale}" />
-      </geometry>
-      <xacro:black_material />
-    </visual>
-  </link>
-  <link name="oled_screen_link">
-    <visual>
-      <origin xyz="${position_screen}" rpy="0 0 ${pi/2}" />
-      <geometry>
-        <mesh filename="package://waver_description/meshes/oled_screen_link.stl" scale="${scale}" />
-      </geometry>
-      <xacro:dark_blue_material />
-    </visual>
-  </link>
-  <link name="wheel_back_left_link">
-    <inertial>
-      <mass value="${mass_wbl}" />
-      <origin xyz="0 0 0" rpy="0 0 ${pi/2}" />
-      <inertia ixx="6.689307761499951e-05" iyy="4.2676101388344066e-05" izz="4.2578787253633605e-05"
-        ixy="0.0" iyz="0.0" ixz="0.0" />
-    </inertial>
-    <visual>
-      <origin xyz="${position_wbl}" rpy="0 0 ${pi/2}" />
-      <geometry>
-        <mesh filename="package://waver_description/meshes/wheel_back_left_link.stl"
-          scale="${scale}" />
-      </geometry>
-      <xacro:black_material />
-    </visual>
-    <collision>
-      <origin xyz="0 0 0" rpy="${pi/2} 0 0" />
-      <geometry>
-        <cylinder radius="${wheel_radius}" length="${wheel_width}" />
-      </geometry>
-    </collision>
-  </link>
-  <link name="wheel_front_left_link">
-    <inertial>
-      <mass value="${mass_wfl}" />
-      <origin xyz="0 0 0" rpy="0 0 ${pi/2}" />
-      <inertia ixx="6.6894731155928e-05" iyy="4.2676101388344066e-05" izz="4.2580440794562095e-05"
-        ixy="0.0" iyz="0.0" ixz="0.0" />
-    </inertial>
-    <visual>
-      <origin xyz="${position_wfl}" rpy="0 0 ${pi/2}" />
-      <geometry>
-        <mesh filename="package://waver_description/meshes/wheel_front_left_link.stl"
-          scale="${scale}" />
-      </geometry>
-      <xacro:black_material />
-    </visual>
-    <collision>
-      <origin xyz="0 0 0" rpy="${pi/2} 0 0" />
-      <geometry>
-        <cylinder radius="${wheel_radius}" length="${wheel_width}" />
-      </geometry>
-    </collision>
-  </link>
-  <link name="wheel_front_right_link">
-    <inertial>
-      <mass value="${mass_wfr}" />
-      <origin xyz="0 0 0" rpy="0 0 ${pi/2}" />
-      <inertia ixx="6.689307761499951e-05" iyy="4.267610303653357e-05" izz="4.2578788901823125e-05"
-        ixy="0.0" iyz="0.0" ixz="0.0" />
-    </inertial>
-    <visual>
-      <origin xyz="${position_wfr}" rpy="0 0 ${pi/2}" />
-      <geometry>
-        <mesh filename="package://waver_description/meshes/wheel_front_right_link.stl"
-          scale="${scale}" />
-      </geometry>
-      <xacro:black_material />
-    </visual>
-    <collision>
-      <origin xyz="0 0 0" rpy="${pi/2} 0 0" />
-      <geometry>
-        <cylinder radius="${wheel_radius}" length="${wheel_width}" />
-      </geometry>
-    </collision>
-  </link>
-  <link name="wheel_back_right_link">
-    <inertial>
-      <mass value="${mass_wbr}" />
-      <origin xyz="0 0 0" rpy="0 0 ${pi/2}" />
-      <inertia ixx="6.6894731155928e-05" iyy="4.267610303653357e-05" izz="4.25804424427516e-05"
-        ixy="0.0" iyz="0.0" ixz="0.0" />
-    </inertial>
-    <visual>
-      <origin xyz="${position_wbr}" rpy="0 0 ${pi/2}" />
-      <geometry>
-        <mesh filename="package://waver_description/meshes/wheel_back_right_link.stl"
-          scale="${scale}" />
-      </geometry>
-      <xacro:black_material />
-    </visual>
-    <collision>
-      <origin xyz="0 0 0" rpy="${pi/2} 0 0" />
-      <geometry>
-        <cylinder radius="${wheel_radius}" length="${wheel_width}" />
-      </geometry>
-    </collision>
-  </link>
-  <!-- ******************************* Links ******************************* -->
-  <joint
-    name="base_joint" type="fixed">
-    <origin xyz="0.0 0.0 33.7e-3" rpy="0 0 0" />
-    <parent link="base_footprint" />
-    <child link="base_link" />
-  </joint>
-  <joint name="base_top_joint" type="fixed">
-    <origin xyz="0 0 0" rpy="0 0 0" />
-    <parent link="base_link" />
-    <child link="top_shell_link" />
-  </joint>
-  <joint name="top_acces_joint" type="fixed">
-    <origin xyz="${positions_acces_joint}" rpy="0 0 0" />
-    <parent link="top_shell_link" />
-    <child link="accessories_link" />
-  </joint>
-  <joint name="top_acces1_joint" type="fixed">
-    <origin xyz="${positions_acces1_joint}" rpy="0 0 0" />
-    <parent link="top_shell_link" />
-    <child link="accessories1_link" />
-  </joint>
-  <joint name="top_screen_joint" type="fixed">
-    <origin xyz="${positions_screen_joint}" rpy="0 0 0" />
-    <parent link="top_shell_link" />
-    <child link="oled_screen_link" />
-  </joint>
-  <joint name="wheel_back_left_joint" type="continuous">
-    <origin xyz="${position_wbl_joint}" rpy="0 0 0" />
-    <parent link="base_link" />
-    <child link="wheel_back_left_link" />
-    <axis xyz="0 1 0" />
-  </joint>
-  <joint name="wheel_front_left_joint" type="continuous">
-    <origin xyz="${position_wfl_joint}" rpy="0 0 0" />
-    <parent link="base_link" />
-    <child link="wheel_front_left_link" />
-    <axis xyz="0 1 0" />
-  </joint>
-  <joint name="wheel_front_right_joint" type="continuous">
-    <origin xyz="${position_wfr_joint}" rpy="0 0 0" />
-    <parent link="base_link" />
-    <child link="wheel_front_right_link" />
-    <axis xyz="0 1 0" />
-  </joint>
-  <joint name="wheel_back_right_joint" type="continuous">
-    <origin xyz="${position_wbr_joint}" rpy="0 0 0" />
-    <parent link="base_link" />
-    <child link="wheel_back_right_link" />
-    <axis xyz="0 1 0" />
-  </joint>
+      <origin xyz="0 0 0"/>
+      <geometry><box size="0.020 0.020 0.004"/></geometry>
+      <material name="green"/>
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