Commit message: cmd vel upravy a tak

File: gazebo/waver_sim/description/lidar.xacro (robot description, xacro)
@@ -25,5 +25,5 @@
   </link>
   <joint name="lidar_joint" type="fixed">
-    <origin xyz="0.04 0 0.092" rpy="0 0 0"/>
+    <origin xyz="-0.04 0 0.092" rpy="0 0 0"/>
     <parent link="base_link"/>
     <child  link="lidar_link"/>
